File: kicad/macpro62-backplane-v2/backplane.kicad_pcb (KiCad board)
At the start: 4 copper layers, 122 x 122 mm, 152 parts, among them J1 ME1022410103011 Mini Cool Edg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, J10 MCIO 124P RA (C4867471) -> Fa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, J2 Molex 43045-0812 Micro-Fit 2x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, J3 BM15B-GHS-TBT (C5305069) Face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, J4 BM15B-GHS-TBT (C5305069) Face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, J6 BM15B-GHS-TBT (C5305069) IOB-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, J7 M.2 M-key socket LOTES APCI01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, J8 BM03B-SRSS-TB SWD (DNP), J9 MCIO 124P RA G97R24332HR clas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, Q1 AO3401A P-MOS, Q10 2N7002 N-MOS, Q11 2N7002 N-MOS, Q2 AO3401A P-MOS, Q3 AO3401A P-MOS, Q4 2N7002 N-MOS, Q5 AO3401A P-MOS, Q6 AO3401A P-MOS, Q7 AO3401A P-MOS, Q8 AO3401A P-MOS, Q9 2N7002 N-MOS, SW1 BOOTSEL (TS-1187A), SW2 BENCH power button (TS-1187A), U1 RP2350B QFN-80 (C42415655), U2 W25Q128JVSIQ (C97521, basic), U3 TMP1075DGKR @0x48 core side (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, U4 TMP1075DGKR @0x49 PSU side (C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, U5 INA226AIDGSR @0x40 (C49851), U6 TPS563201DDCR (C116592) -> 3V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, U7 TPS563201DDCR (C116592) -> 5V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, U8 SN74LVC1G74DCUR thermal latch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, Y1 12MHz 3225 crystal 20pF

Commit message: Fix KiCad 9 rule files: add mm units (whole file was rejected)
KiCad 9.0.2 rejects any .kicad_dru with unitless numbers, so the custom
rules never applied to DRC or zone fills on the base board (A1/A2/v3),
SSD 2x and the I/O modules.

- Base board A1/A2/v3, SSD 2x: pour rule in mm, applied to tracks only.
  Refilled; pours now hold 0.5 mm from 85R and 0.4 mm from 90R pairs
  (were 0.2 mm). Added J7 pad 45 GND stub + via; restored the 3V3_SB
  L3 link to Q2/R34 (A1/A2). JLC gerbers/drill regenerated; BOM/CPL unchanged.
- I/O modules and panels: rules in mm; diff-pair gap check exempts
  connector/test-point breakouts and T/* TDR coupons. No copper change.
- Rule generators (make_pro.py, build_modules.py) updated to match.
DRC: 0 errors, 0 unconnected on all boards.
Routing:
- net GND: track 358.4 -> 359.2 mm, vias 611 -> 612
Changed lines of the file:
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@@
 	)
 	(segment
+		(start 124.7 131.75)
+		(end 123.95 131.75)
+		(width 0.2)
+		(layer "F.Cu")
+		(net 2)
+	)
+	(segment
 		(start 154.005382 48.014719)
 		(end 155.067095 46.629875)
@@
 	)
 	(via
+		(at 123.95 131.75)
+		(size 0.45)
+		(drill 0.25)
+		(layers "F.Cu" "B.Cu")
+		(net 2)
+	)
+	(via
 		(at 132 97)
 		(size 0.45)
@@
 		(width 0.2)
 		(layer "In2.Cu")
+		(net 115)
+	)
+	(segment
+		(start 131.85 122.35)
+		(end 132.05 122.1)
+		(width 0.2)
+		(layer "In2.Cu")
