File: boards/base-v3/kicad/backplane.kicad_pcb (KiCad board)
At the start: 6 copper layers, 122 x 122 mm, 233 parts, among them J1 ME1022410103011 Mini Cool Edg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, J11 MEG300 84501 GPU face (pinout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, J12 MEG300 84501 SSD face (base-s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, J2 Molex 43045-0812 Micro-Fit 2x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, J3 BM15B-GHS-TBT (C5305069) Face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, J4 BM15B-GHS-TBT (C5305069) Face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, J6 BM15B-GHS-TBT (C5305069) IOB-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, J7 M.2 M-key socket LOTES APCI01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, J8 BM03B-SRSS-TB SWD (DNP), Q1 AO3401A P-MOS, Q10 2N7002 N-MOS, Q11 2N7002 N-MOS, Q12 2N7002 N-MOS, Q2 AO3401A P-MOS, Q3 AO3401A P-MOS, Q4 2N7002 N-MOS, Q5 AO3401A P-MOS, Q6 AO3401A P-MOS, Q7 AO3401A P-MOS, Q8 AO3401A P-MOS, Q9 2N7002 N-MOS, SW1 BOOTSEL (TS-1187A), SW2 BENCH power button (TS-1187A), U1 RP2350B QFN-80 (C42415655), U2 W25Q128JVSIQ (C97521, basic), U20 DS320PR1601ZDGR, U21 DS320PR810NJXR, U22 DS320PR810NJXR, U23 PT5161L_ALT_DNP, U24 TPS565208DDCR, U25 TPS259824LNRGE, U26 TMP1075DGKR @0x4A core side (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, U3 TMP1075DGKR @0x48 core side (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, U4 TMP1075DGKR @0x49 PSU side (C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, U5 INA226AIDGSR @0x40 (C49851), U6 TPS563201DDCR (C116592) -> 3V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, U7 TPS563201DDCR (C116592) -> 5V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, U8 SN74LVC1G74DCUR thermal latch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, Y1 12MHz 3225 crystal 20pF

Commit message: Sync design state 2026-10-29: J1 v4 pinned, boot drive dropped, no NDA parts, base board J13/J14 and fab push, SSD/I/O power and pinmaps
Parts:
- removed C17: 22uF 25V X5R 0805, MP62_BP:C_0805_2012Metric
- removed C18: 100nF 16V X7R 0402, MP62_BP:C_0402_1005Metric
- removed D2: SS34 3A 40V Schottky SMA, MP62_BP:D_SMA
- removed D9: LED red 0603, MP62_BP:LED_0603_1608Metric
- removed J2: Molex 43045-0812 Micro-Fit 2x4 (C277661), MP62_BP:Molex_Micro-Fit_3.0_43045-0812_2x04_P3.00mm_Vertical
- removed J6: BM15B-GHS-TBT (C5305069) IOB-LINK, MP62_BP:JST_GH_BM15B-GHS-TBT_1x15-1MP_P1.25mm_Vertical
- removed J7: M.2 M-key socket LOTES APCI0107 class (C841661) - DNP optio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, MP62_BP:MP62_M2_MKey_SMT_H4.2_PLACEHOLDER
- removed Q3: AO3401A P-MOS, MP62_BP:SOT-23
- removed Q4, Q9: 2N7002 N-MOS, MP62_BP:SOT-23
- removed R10, R9: 10k 1% 0402, MP62_BP:R_0402_1005Metric
- removed R54: 1k 1% 0402, MP62_BP:R_0402_1005Metric
- removed U23: PT5161L_ALT_DNP, MP62_BP:Astera_PT5161L_ALT_DNP_PLACEHOLDER
- added C84: 100nF 16V X7R 0402, MP62_BP:C_0402_1005Metric, B.Cu at (145.7, 141.5)
- added J13: MEG300 84501 I/O face (base-iob-megarray.csv), MP62_BP:Amphenol_MegArray_84501_300P_10x30_P1.27mm_UNVERIFIED, F.Cu at (148.9, 146.8)
- added J14: MCIO 124P RA (C4867471) -> Face S x4 + x2 (v3 slot B; lanes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, MP62_MCIO_124P_Vertical_SMT_TE2360189_PLACEHOLDER, F.Cu at (150.0, 130.0)
- added R127: 10k 1% 0402, MP62_BP:R_0402_1005Metric, B.Cu at (154.4, 141.5)
- added R128: 10k 1% 0402, MP62_BP:R_0402_1005Metric, B.Cu at (154.4, 143.0)
- added R129: 10k 1% 0402, MP62_BP:R_0402_1005Metric, B.Cu at (154.4, 139.8)
- added U27: TSSOP-16, MP62_BP:TSSOP-16_4.4x5mm_P0.65mm, B.Cu at (150.1, 141.7)
- R122: value 249R 1% 0402 (ILIM ~6.0 A typ, SLVSEI3D p.9: 300R=4.98 A, 182R=8.13 A) -> 300R 1% 0402 (ILIM ~5.0 A)
- moved C39 41.8 mm to (115.5, 132.9)
- moved R46 35.2 mm to (108.3, 120.1), turned to 180 degrees
- moved C37 34.2 mm to (113.2, 134.8)
- moved R60 32.2 mm to (113.8, 132.9), turned to 180 degrees
- moved C79 32.1 mm to (158.6, 97.9)
- moved R121 30.7 mm to (131.4, 65.8), turned to 90 degrees
- moved D5 29.6 mm to (151.0, 104.7)
- moved R8 28.5 mm to (118.5, 126.2), turned to 90 degrees
- moved J8 28.2 mm to (113.2, 138.8), turned to 180 degrees
- moved D1 28.0 mm to (125.0, 124.7)
- moved R51 27.9 mm to (117.5, 117.0), turned to 180 degrees
- moved Q6 27.0 mm to (125.4, 118.8)
- moved R13 26.6 mm to (127.9, 137.5)
- moved R63 25.7 mm to (122.5, 117.8), turned to 180 degrees
- moved Q7 25.3 mm to (180.2, 145.7)
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Connections:
- J1 pad A101: FS_TX6_P -> GND
- J1 pad A102: FS_TX6_N -> EFUSE_IN
- J1 pad A103: GND -> EFUSE_IN
- J1 pad A104: unconnected-(J1-RSTBTN#-PadA104) -> EFUSE_IN
- J1 pad A105: CB_PWR_ALERT_N -> EFUSE_IN
- J1 pad A106: GND -> EFUSE_IN
- J1 pad A107: 5V_SBY -> EFUSE_IN
- J1 pad A108: 5V_SBY -> GND
- J1 pad A110: 5V_SBY -> GND
- J1 pad A111: 5V_SBY -> GND
- J1 pad A54: FS_TX7_P -> FS_TX0_P
- J1 pad A55: FS_TX7_N -> FS_TX0_N
- J1 pad A57: GND -> FS_TX1_P
- J1 pad A58: FS_TX3_P -> FS_TX1_N
- J1 pad A59: FS_TX3_N -> GND
- J1 pad A60: GND -> FS_TX2_P
- J1 pad A61: FS_TX2_P -> FS_TX2_N
- J1 pad A62: FS_TX2_N -> GND
- J1 pad A63: GND -> FS_TX3_P
- J1 pad A64: FS_TX1_P -> FS_TX3_N
- J1 pad A65: FS_TX1_N -> GND
- J1 pad A66: GND -> FS_TX4_P
- J1 pad A67: FS_TX0_P -> FS_TX4_N
- J1 pad A68: FS_TX0_N -> GND
- J1 pad A69: GND -> FS_TX5_P
- J1 pad A70: FS_REFCLK_P -> FS_TX5_N
- J1 pad A71: FS_REFCLK_N -> GND
- J1 pad A72: GND -> FS_TX6_P
- J1 pad A73: SATA0_TX_P -> FS_TX6_N
- J1 pad A74: SATA0_TX_N -> GND
- J1 pad A75: GND -> FS_TX7_P
- J1 pad A76: unconnected-(J1-RSVD_HS_A1_P-PadA76) -> FS_TX7_N
- J1 pad A77: unconnected-(J1-RSVD_HS_A1_N-PadA77) -> GND
- J1 pad A78: GND -> FS_REFCLK_P
- J1 pad A79: unconnected-(J1-RSVD_HS_A2_P-PadA79) -> FS_REFCLK_N
- J1 pad A80: unconnected-(J1-RSVD_HS_A2_N-PadA80) -> GND
- J1 pad A81: GND -> USB2_MCU_P
- J1 pad A82: FS_TX4_P -> USB2_MCU_N
- J1 pad A83: FS_TX4_N -> CB_SUS_S3_N
- J1 pad A84: GND -> CB_SUS_S45_N
- J1 pad A85: GND -> CB_RSMRST_N
- J1 pad A86: FS_TX5_P -> CB_VIN_PWR_OK
- J1 pad A87: FS_TX5_N -> CB_PLTRST_N
- J1 pad A88: GND -> CB_THERMTRIP_N
- J1 pad A89: CB_SUS_S3_N -> CB_CARRIER_HOT_N
- J1 pad A90: CB_SUS_S45_N -> CB_WAKE_N
- J1 pad A91: GND -> unconnected-(J1-GND-PadA91)
- J1 pad A92: CB_RSMRST_N -> GND
- J1 pad A93: CB_VIN_PWR_OK -> 3V3_SB
- J1 pad A94: GND -> 5V_SBY
- J1 pad A95: CB_PLTRST_N -> 5V_SBY
- J1 pad A96: CB_THERMTRIP_N -> 5V_SBY
- J1 pad A98: CB_CARRIER_HOT_N -> GND
- J1 pad A99: CB_WAKE_N -> GND
- J1 pad B101: FS_REFCLK1_P -> GND
- J1 pad B102: FS_REFCLK1_N -> EFUSE_IN
- J1 pad B103: GND -> EFUSE_IN
- J1 pad B104: FS_RX6_N -> EFUSE_IN
- J1 pad B105: FS_RX6_P -> EFUSE_IN
- J1 pad B106: GND -> EFUSE_IN
- J1 pad B107: 3V3_SB -> EFUSE_IN
- J1 pad B108: 3V3_SB -> GND
- J1 pad B110: 5V_SBY -> GND
- J1 pad B111: 5V_SBY -> GND
- J1 pad B54: FS_RX7_P -> FS_RX0_P
- J1 pad B55: FS_RX7_N -> FS_RX0_N
- J1 pad B57: GND -> FS_RX1_P
- J1 pad B58: FS_RX3_P -> FS_RX1_N
- J1 pad B59: FS_RX3_N -> GND
- J1 pad B60: GND -> FS_RX2_P
- J1 pad B61: FS_RX2_P -> FS_RX2_N
- J1 pad B62: FS_RX2_N -> GND
- J1 pad B63: GND -> FS_RX3_P
- J1 pad B64: FS_RX1_P -> FS_RX3_N
- J1 pad B65: FS_RX1_N -> GND
- J1 pad B66: GND -> FS_RX4_P
- J1 pad B67: FS_RX0_P -> FS_RX4_N
- J1 pad B68: FS_RX0_N -> GND
- J1 pad B69: GND -> FS_RX5_P
- J1 pad B70: SATA0_RX_P -> FS_RX5_N
- J1 pad B71: SATA0_RX_N -> GND
- J1 pad B72: GND -> FS_RX6_P
- J1 pad B73: USB2_MCU_P -> FS_RX6_N
- J1 pad B74: USB2_MCU_N -> GND
- J1 pad B75: GND -> FS_RX7_P
- J1 pad B76: USB2_FACES_P -> FS_RX7_N
- J1 pad B77: USB2_FACES_N -> GND
- J1 pad B78: GND -> FS_REFCLK1_P
- J1 pad B79: USB2_SPARE_P -> FS_REFCLK1_N
- J1 pad B80: USB2_SPARE_N -> GND
- J1 pad B82: FS_RX4_P -> GND
- J1 pad B83: FS_RX4_N -> GND
- J1 pad B84: GND -> CB_I2C0_SCL
- J1 pad B85: GND -> CB_I2C0_SDA
- J1 pad B86: FS_RX5_N -> CB_UART0_TX
- J1 pad B87: FS_RX5_P -> CB_UART0_RX
- J1 pad B88: GND -> CB_FAN_PWM
- J1 pad B89: unconnected-(J1-BIOS_SEL-PadB89) -> CB_FAN_TACH
- J1 pad B90: CB_I2C0_SCL -> GND
- J1 pad B91: GND -> CB_PWR_ALERT_N
- J1 pad B92: CB_I2C0_SDA -> GND
- J1 pad B93: CB_UART0_TX -> 3V3_SB
- J1 pad B94: GND -> 5V_SBY
- J1 pad B95: CB_UART0_RX -> 5V_SBY
- J1 pad B96: CB_FAN_PWM -> 5V_SBY
- J1 pad B98: CB_FAN_TACH -> GND
- J1 pad B99: CB_PWRBTN_N -> GND
- J12 pad J1: 12V_MAIN_IN -> GND
- J12 pad J10: 12V_MAIN_IN -> GND
- J12 pad J11: 12V_MAIN_IN -> GND
- J12 pad J12: 12V_MAIN_IN -> GND
- J12 pad J2: 12V_MAIN_IN -> GND
- J12 pad J3: 12V_MAIN_IN -> GND
- J12 pad J4: 12V_MAIN_IN -> GND
- J12 pad J5: 12V_MAIN_IN -> GND
- J12 pad J6: 12V_MAIN_IN -> GND
- J12 pad J7: 12V_MAIN_IN -> GND
- J12 pad J8: 12V_MAIN_IN -> GND
- J12 pad J9: 12V_MAIN_IN -> GND
- U1 pad 20: PSU_PWR_OK_M -> CB_SMB_ALERT_N
- U1 pad 47: FP_MCIO_PRSNT_N -> I2C_BB_SCL
- U1 pad 8: FS_MCIO_PRSNT_N -> I2C_BB_SDA
- U20 pad AA29: FP_RX1_N_A -> FP_RX1_N
- U20 pad AB1: FP_TX1_N_A -> FP_TX1_N
- U20 pad AF26: FP_RX2_P_A -> FP_RX2_P
- U20 pad AG2: FP_TX2_N_A -> FP_TX2_N
- U20 pad AH29: FP_RX2_N_A -> FP_RX2_N
- U20 pad AJ1: FP_TX2_P_A -> FP_TX2_P
- U20 pad AN26: FP_RX3_P_A -> FP_RX3_P
- U20 pad AP2: FP_TX3_N_A -> FP_TX3_N
- U20 pad AR29: FP_RX3_N_A -> FP_RX3_N
- U20 pad AT1: FP_TX3_P_A -> FP_TX3_P
- U20 pad AY26: FP_RX4_P_A -> FP_RX4_P
- U20 pad BA2: FP_TX4_P_A -> FP_TX4_P
- U20 pad BB29: FP_RX4_N_A -> FP_RX4_N
- U20 pad BC1: FP_TX4_N_A -> FP_TX4_N
- U20 pad BG26: FP_RX5_P_A -> FP_RX5_P
- U20 pad BH2: FP_TX5_P_A -> FP_TX5_P
- U20 pad BJ29: FP_RX5_N_A -> FP_RX5_N
- U20 pad BK1: FP_TX5_N_A -> FP_TX5_N
- U20 pad BP26: FP_RX6_P_A -> FP_RX6_P
- U20 pad BR2: FP_TX6_N_A -> FP_TX6_N
- U20 pad BT29: FP_RX6_N_A -> FP_RX6_N
- U20 pad BU1: FP_TX6_P_A -> FP_TX6_P
- U20 pad CA26: FP_RX7_P_A -> FP_RX7_P
- U20 pad CB2: FP_TX7_N_A -> FP_TX7_N
- U20 pad CC29: FP_RX7_N_A -> FP_RX7_N
- U20 pad CD1: FP_TX7_P_A -> FP_TX7_P
- U20 pad CH26: FP_RX8_P_A -> FP_RX8_P
- U20 pad CJ2: FP_TX8_P_A -> FP_TX8_P
- U20 pad CK29: FP_RX8_N_A -> FP_RX8_N
- U20 pad CL1: FP_TX8_N_A -> FP_TX8_N
- U20 pad CR26: FP_RX9_P_A -> FP_RX9_P
- U20 pad CT2: FP_TX9_P_A -> FP_TX9_P
- U20 pad CU29: FP_RX9_N_A -> FP_RX9_N
- U20 pad CV1: FP_TX9_N_A -> FP_TX9_N
- U20 pad DB26: FP_RX10_P_A -> FP_RX10_P
- U20 pad DC2: FP_TX10_N_A -> FP_TX10_N
- U20 pad DD29: FP_RX10_N_A -> FP_RX10_N
- U20 pad DE1: FP_TX10_P_A -> FP_TX10_P
- U20 pad DJ26: FP_RX11_P_A -> FP_RX11_P
- U20 pad DK2: FP_TX11_N_A -> FP_TX11_N
- U20 pad DL29: FP_RX11_N_A -> FP_RX11_N
- U20 pad DM1: FP_TX11_P_A -> FP_TX11_P
- U20 pad DT26: FP_RX12_P_A -> FP_RX12_P
- U20 pad DU2: FP_TX12_P_A -> FP_TX12_P
- U20 pad DV29: FP_RX12_N_A -> FP_RX12_N
- U20 pad DW1: FP_TX12_N_A -> FP_TX12_N
- U20 pad EC26: FP_RX13_P_A -> FP_RX13_P
- U20 pad ED2: FP_TX13_P_A -> FP_TX13_P
- U20 pad EE29: FP_RX13_N_A -> FP_RX13_N
- U20 pad EF1: FP_TX13_N_A -> FP_TX13_N
- U20 pad EK26: FP_RX14_P_A -> FP_RX14_P
- U20 pad EL2: FP_TX14_N_A -> FP_TX14_N
- U20 pad EM29: FP_RX14_N_A -> FP_RX14_N
- U20 pad EN1: FP_TX14_P_A -> FP_TX14_P
- U20 pad EU26: FP_RX15_P_A -> FP_RX15_P
- U20 pad EV2: FP_TX15_N_A -> FP_TX15_N
- U20 pad EW29: FP_RX15_N_A -> FP_RX15_N
- U20 pad EY1: FP_TX15_P_A -> FP_TX15_P
- U20 pad M26: FP_RX0_P_A -> FP_RX0_P
- U20 pad N2: FP_TX0_P_A -> FP_TX0_P
- U20 pad P29: FP_RX0_N_A -> FP_RX0_N
- U20 pad R1: FP_TX0_N_A -> FP_TX0_N
- U20 pad W26: FP_RX1_P_A -> FP_RX1_P
- U20 pad Y2: FP_TX1_P_A -> FP_TX1_P
- U21 pad 1: FS_TX0_P_A -> FS_TX0_P
- U21 pad 10: FS_TX3_P_A -> FS_TX3_P
- U21 pad 11: FS_TX3_N_A -> FS_TX3_N
- U21 pad 2: FS_TX0_N_A -> FS_TX0_N
- U21 pad 33: FS_RX3_N_A -> FS_RX3_N
- U21 pad 34: FS_RX3_P_A -> FS_RX3_P
- U21 pad 36: FS_RX2_N_A -> FS_RX2_N
- U21 pad 37: FS_RX2_P_A -> FS_RX2_P
- U21 pad 39: FS_RX1_N_A -> FS_RX1_N
- U21 pad 4: FS_TX1_P_A -> FS_TX1_P
- U21 pad 40: FS_RX1_P_A -> FS_RX1_P
- U21 pad 42: FS_RX0_N_A -> FS_RX0_N
- U21 pad 43: FS_RX0_P_A -> FS_RX0_P
- U21 pad 5: FS_TX1_N_A -> FS_TX1_N
- U21 pad 7: FS_TX2_P_A -> FS_TX2_P
- U21 pad 8: FS_TX2_N_A -> FS_TX2_N
- U22 pad 1: FS_TX4_P_A -> FS_TX4_P
- U22 pad 10: FS_TX7_P_A -> FS_TX7_P
- U22 pad 11: FS_TX7_N_A -> FS_TX7_N
- U22 pad 2: FS_TX4_N_A -> FS_TX4_N
- U22 pad 33: FS_RX7_N_A -> FS_RX7_N
- U22 pad 34: FS_RX7_P_A -> FS_RX7_P
- U22 pad 36: FS_RX6_N_A -> FS_RX6_N
- U22 pad 37: FS_RX6_P_A -> FS_RX6_P
- U22 pad 39: FS_RX5_N_A -> FS_RX5_N
- U22 pad 4: FS_TX5_P_A -> FS_TX5_P
- U22 pad 40: FS_RX5_P_A -> FS_RX5_P
- U22 pad 42: FS_RX4_N_A -> FS_RX4_N
- U22 pad 43: FS_RX4_P_A -> FS_RX4_P
- U22 pad 5: FS_TX5_N_A -> FS_TX5_N
- U22 pad 7: FS_TX6_P_A -> FS_TX6_P
- U22 pad 8: FS_TX6_N_A -> FS_TX6_N
Routing:
- net GND: track 361.5 -> 0.00 mm, vias 566 -> 0
- net 3V3_SB: track 210.7 -> 0.00 mm, vias 85 -> 0
- net 3V3_AUX_S: track 205.6 -> 0.00 mm, vias 20 -> 0
- net FP_MCIO_PRSNT_N: track 176.8 -> 0.00 mm, vias 4 -> 0
- net FP_THERM_ALERT_N: track 155.8 -> 0.00 mm, vias 11 -> 0
- net 5V_SBY: track 154.5 -> 0.00 mm, vias 15 -> 0
- net I2C_SYS_SDA: track 149.1 -> 0.00 mm, vias 10 -> 0
- net FS_SMB_ALERT_N: track 147.6 -> 0.00 mm, vias 9 -> 0
- net I2C_SYS_SCL: track 138.5 -> 0.00 mm, vias 5 -> 0
- net FS_THERM_ALERT_N: track 136.0 -> 0.00 mm, vias 4 -> 0
- net PWRBTN_IN_N: track 133.3 -> 0.00 mm, vias 6 -> 0
- net FP_PWR_GOOD: track 133.0 -> 0.00 mm, vias 10 -> 0
- net BP_OTEMP_N: track 129.0 -> 0.00 mm, vias 4 -> 0
- net SYS_INT_N: track 124.1 -> 0.00 mm, vias 2 -> 0
- net FP_PRSNT_N: track 123.6 -> 0.00 mm, vias 2 -> 0
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