File: boards/base-v3/kicad/backplane.kicad_sch (KiCad schematic)
At the start: 235 parts, among them J1 ME1022410103011 Mini Cool Edg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, J10 MCIO 124P RA (C4867471) -> Fa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, J11 MEG300 84501 GPU face (pinout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, J12 MEG300 84501 SSD face, J2 Molex 43045-0812 Micro-Fit 2x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, J3 BM15B-GHS-TBT (C5305069) Face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, J4 BM15B-GHS-TBT (C5305069) Face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, J6 BM15B-GHS-TBT (C5305069) IOB-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, J7 M.2 M-key socket LOTES APCI01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, J8 BM03B-SRSS-TB SWD (DNP), J9 MCIO 124P RA G97R24332HR clas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, Q1 AO3401A P-MOS, Q10 2N7002 N-MOS, Q11 2N7002 N-MOS, Q12 2N7002 N-MOS, Q2 AO3401A P-MOS, Q3 AO3401A P-MOS, Q4 2N7002 N-MOS, Q5 AO3401A P-MOS, Q6 AO3401A P-MOS, Q7 AO3401A P-MOS, Q8 AO3401A P-MOS, Q9 2N7002 N-MOS, SW1 BOOTSEL (TS-1187A), SW2 BENCH power button (TS-1187A), U1 RP2350B QFN-80 (C42415655), U2 W25Q128JVSIQ (C97521, basic), U20 DS320PR1601ZDGR, U21 DS320PR810NJXR, U22 DS320PR810NJXR, U23 PT5161L_ALT_DNP, U24 TPS565208DDCR, U25 TPS259824LNRGE, U26 TMP1075DGKR @0x4A U20 redrive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, U3 TMP1075DGKR @0x48 core side (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, U4 TMP1075DGKR @0x49 PSU side (C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, U5 INA226AIDGSR @0x40 (C49851), U6 TPS563201DDCR (C116592) -> 3V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, U7 TPS563201DDCR (C116592) -> 5V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, U8 SN74LVC1G74DCUR thermal latch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, Y1 12MHz 3225 crystal 20pF

Commit message: Sync design state 2026-10-29: J1 v4 pinned, boot drive dropped, no NDA parts, base board J13/J14 and fab push, SSD/I/O power and pinmaps
Parts:
- removed C17: 22uF 25V X5R 0805, MP62_BP:C_0805_2012Metric, symbol MP62_BP:C
- removed C18: 100nF 16V X7R 0402, MP62_BP:C_0402_1005Metric, symbol MP62_BP:C
- removed D2: SS34 3A 40V Schottky SMA, MP62_BP:D_SMA, symbol MP62_BP:D
- removed D9: LED red 0603, MP62_BP:LED_0603_1608Metric, symbol MP62_BP:LED
- removed J10: MCIO 124P RA (C4867471) -> Face S x4 + slot B x4 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, MP62_BP:MP62_MCIO_124P_RA_SFF-TA-1016, symbol MP62_BP:MCIO124_BP
- removed J2: Molex 43045-0812 Micro-Fit 2x4 (C277661), MP62_BP:Molex_Micro-Fit_3.0_43045-0812_2x04_P3.00mm_Vertical, symbol MP62_BP:MICROFIT8
- removed J6: BM15B-GHS-TBT (C5305069) IOB-LINK, MP62_BP:JST_GH_BM15B-GHS-TBT_1x15-1MP_P1.25mm_Vertical, symbol MP62_BP:GH15_IOB
- removed J7: M.2 M-key socket LOTES APCI0107 class (C841661) -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, MP62_BP:MP62_M2_MKey_SMT_H4.2_PLACEHOLDER, symbol MP62_BP:M2_M_SATA
- removed J9: MCIO 124P RA G97R24332HR class (C4867471, 0 stock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, MP62_BP:MP62_MCIO_124P_RA_SFF-TA-1016, symbol MP62_BP:MCIO124_BP
- removed Q3, Q7, Q8: AO3401A P-MOS, MP62_BP:SOT-23, symbol MP62_BP:PMOS
- removed Q4, Q9: 2N7002 N-MOS, MP62_BP:SOT-23, symbol MP62_BP:NMOS
- removed R10, R15, R9: 10k 1% 0402, MP62_BP:R_0402_1005Metric, symbol MP62_BP:R
- removed R12, R55: 100k 1% 0402, MP62_BP:R_0402_1005Metric, symbol MP62_BP:R
- removed R54: 1k 1% 0402, MP62_BP:R_0402_1005Metric, symbol MP62_BP:R
- removed U23: PT5161L_ALT_DNP, MP62_BP:Astera_PT5161L_ALT_DNP_PLACEHOLDER, symbol MP62_BP:PT5161L_ALT
- added C84: 100nF 16V X7R 0402, MP62_BP:C_0402_1005Metric, symbol MP62_BP:C
- added J13: MEG300 84501 I/O face (base-iob-megarray.csv), MP62_BP:Amphenol_MegArray_84501_300P_10x30_P1.27mm_UNVERIFIED, symbol MP62_BP:MEG300
- added J14: MCIO 124P RA (C4867471) base end of CPU-board J3 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, MP62_Placeholders:MP62_MCIO_124P_Vertical_SMT_TE2360189_PLACEHOLDER, symbol MP62_BP:MCIO124_BP
- added R127: 10k 1% 0402 (IOB_PLT_RST_N pull-down: reset asser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, MP62_BP:R_0402_1005Metric, symbol MP62_BP:R
- added R128: 10k 1% 0402 (IOB USB OC# A pull-up), MP62_BP:R_0402_1005Metric, symbol MP62_BP:R
- added R129: 10k 1% 0402 (IOB USB OC# C pull-up), MP62_BP:R_0402_1005Metric, symbol MP62_BP:R
- added U27: TCA6408APWR I2C GPIO expander @0x20 (IOB sideband), MP62_BP:TSSOP-16_4.4x5mm_P0.65mm, symbol MP62_BP:TCA6408A
- R122: value 249R 1% 0402 (ILIM ~6.0 A typ, SLVSEI3D p.9: 300R=4.98 A, 182R=8.13 A) -> 300R 1% 0402 (ILIM ~5.0 A typ for ~3.5 A load, SLVSEI3D p.9: 300R=4.98 A)
Connections:
- net FP_RX0_N_A is gone; now on net FP_RX0_N: U20.P29 (A_PETn0)
- net FP_RX0_P_A is gone; now on net FP_RX0_P: U20.M26 (A_PETp0)
- net FP_RX10_N_A is gone; now on net FP_RX10_N: U20.DD29 (A_PETn10)
- net FP_RX10_P_A is gone; now on net FP_RX10_P: U20.DB26 (A_PETp10)
- net FP_RX11_N_A is gone; now on net FP_RX11_N: U20.DL29 (A_PETn11)
- net FP_RX11_P_A is gone; now on net FP_RX11_P: U20.DJ26 (A_PETp11)
- net FP_RX12_N_A is gone; now on net FP_RX12_N: U20.DV29 (A_PETn12)
- net FP_RX12_P_A is gone; now on net FP_RX12_P: U20.DT26 (A_PETp12)
- net FP_RX13_N_A is gone; now on net FP_RX13_N: U20.EE29 (A_PETn13)
- net FP_RX13_P_A is gone; now on net FP_RX13_P: U20.EC26 (A_PETp13)
- net FP_RX14_N_A is gone; now on net FP_RX14_N: U20.EM29 (A_PETn14)
- net FP_RX14_P_A is gone; now on net FP_RX14_P: U20.EK26 (A_PETp14)
- net FP_RX15_N_A is gone; now on net FP_RX15_N: U20.EW29 (A_PETn15)
- net FP_RX15_P_A is gone; now on net FP_RX15_P: U20.EU26 (A_PETp15)
- net FP_RX1_N_A is gone; now on net FP_RX1_N: U20.AA29 (A_PETn1)
- net FP_RX1_P_A is gone; now on net FP_RX1_P: U20.W26 (A_PETp1)
- net FP_RX2_N_A is gone; now on net FP_RX2_N: U20.AH29 (A_PETn2)
- net FP_RX2_P_A is gone; now on net FP_RX2_P: U20.AF26 (A_PETp2)
- net FP_RX3_N_A is gone; now on net FP_RX3_N: U20.AR29 (A_PETn3)
- net FP_RX3_P_A is gone; now on net FP_RX3_P: U20.AN26 (A_PETp3)
- net FP_RX4_N_A is gone; now on net FP_RX4_N: U20.BB29 (A_PETn4)
- net FP_RX4_P_A is gone; now on net FP_RX4_P: U20.AY26 (A_PETp4)
- net FP_RX5_N_A is gone; now on net FP_RX5_N: U20.BJ29 (A_PETn5)
- net FP_RX5_P_A is gone; now on net FP_RX5_P: U20.BG26 (A_PETp5)
- net FP_RX6_N_A is gone; now on net FP_RX6_N: U20.BT29 (A_PETn6)
- net FP_RX6_P_A is gone; now on net FP_RX6_P: U20.BP26 (A_PETp6)
- net FP_RX7_N_A is gone; now on net FP_RX7_N: U20.CC29 (A_PETn7)
- net FP_RX7_P_A is gone; now on net FP_RX7_P: U20.CA26 (A_PETp7)
- net FP_RX8_N_A is gone; now on net FP_RX8_N: U20.CK29 (A_PETn8)
- net FP_RX8_P_A is gone; now on net FP_RX8_P: U20.CH26 (A_PETp8)
- net FP_RX9_N_A is gone; now on net FP_RX9_N: U20.CU29 (A_PETn9)
- net FP_RX9_P_A is gone; now on net FP_RX9_P: U20.CR26 (A_PETp9)
- net FP_TX0_N_A is gone; now on net FP_TX0_N: U20.R1 (A_PERn0)
- net FP_TX0_P_A is gone; now on net FP_TX0_P: U20.N2 (A_PERp0)
- net FP_TX10_N_A is gone; now on net FP_TX10_N: U20.DC2 (A_PERn10)
- net FP_TX10_P_A is gone; now on net FP_TX10_P: U20.DE1 (A_PERp10)
- net FP_TX11_N_A is gone; now on net FP_TX11_N: U20.DK2 (A_PERn11)
- net FP_TX11_P_A is gone; now on net FP_TX11_P: U20.DM1 (A_PERp11)
- net FP_TX12_N_A is gone; now on net FP_TX12_N: U20.DW1 (A_PERn12)
- net FP_TX12_P_A is gone; now on net FP_TX12_P: U20.DU2 (A_PERp12)
- net FP_TX13_N_A is gone; now on net FP_TX13_N: U20.EF1 (A_PERn13)
- net FP_TX13_P_A is gone; now on net FP_TX13_P: U20.ED2 (A_PERp13)
- net FP_TX14_N_A is gone; now on net FP_TX14_N: U20.EL2 (A_PERn14)
- net FP_TX14_P_A is gone; now on net FP_TX14_P: U20.EN1 (A_PERp14)
- net FP_TX15_N_A is gone; now on net FP_TX15_N: U20.EV2 (A_PERn15)
- net FP_TX15_P_A is gone; now on net FP_TX15_P: U20.EY1 (A_PERp15)
- net FP_TX1_N_A is gone; now on net FP_TX1_N: U20.AB1 (A_PERn1)
- net FP_TX1_P_A is gone; now on net FP_TX1_P: U20.Y2 (A_PERp1)
- net FP_TX2_N_A is gone; now on net FP_TX2_N: U20.AG2 (A_PERn2)
- net FP_TX2_P_A is gone; now on net FP_TX2_P: U20.AJ1 (A_PERp2)
- net FP_TX3_N_A is gone; now on net FP_TX3_N: U20.AP2 (A_PERn3)
- net FP_TX3_P_A is gone; now on net FP_TX3_P: U20.AT1 (A_PERp3)
- net FP_TX4_N_A is gone; now on net FP_TX4_N: U20.BC1 (A_PERn4)
- net FP_TX4_P_A is gone; now on net FP_TX4_P: U20.BA2 (A_PERp4)
- net FP_TX5_N_A is gone; now on net FP_TX5_N: U20.BK1 (A_PERn5)
- net FP_TX5_P_A is gone; now on net FP_TX5_P: U20.BH2 (A_PERp5)
- net FP_TX6_N_A is gone; now on net FP_TX6_N: U20.BR2 (A_PERn6)
- net FP_TX6_P_A is gone; now on net FP_TX6_P: U20.BU1 (A_PERp6)
- net FP_TX7_N_A is gone; now on net FP_TX7_N: U20.CB2 (A_PERn7)
- net FP_TX7_P_A is gone; now on net FP_TX7_P: U20.CD1 (A_PERp7)
- net FP_TX8_N_A is gone; now on net FP_TX8_N: U20.CL1 (A_PERn8)
- net FP_TX8_P_A is gone; now on net FP_TX8_P: U20.CJ2 (A_PERp8)
- net FP_TX9_N_A is gone; now on net FP_TX9_N: U20.CV1 (A_PERn9)
- net FP_TX9_P_A is gone; now on net FP_TX9_P: U20.CT2 (A_PERp9)
- net FS_RX0_N_A is gone; now on net FS_RX0_N: U21.42 (TX4N)
- net FS_RX0_P_A is gone; now on net FS_RX0_P: U21.43 (TX4P)
- net FS_RX1_N_A is gone; now on net FS_RX1_N: U21.39 (TX5N)
- net FS_RX1_P_A is gone; now on net FS_RX1_P: U21.40 (TX5P)
- net FS_RX2_N_A is gone; now on net FS_RX2_N: U21.36 (TX6N)
- net FS_RX2_P_A is gone; now on net FS_RX2_P: U21.37 (TX6P)
- net FS_RX3_N_A is gone; now on net FS_RX3_N: U21.33 (TX7N)
- net FS_RX3_P_A is gone; now on net FS_RX3_P: U21.34 (TX7P)
- net FS_RX4_N_A is gone; now on net FS_RX4_N: U22.42 (TX4N)
- net FS_RX4_P_A is gone; now on net FS_RX4_P: U22.43 (TX4P)
- net FS_RX5_N_A is gone; now on net FS_RX5_N: U22.39 (TX5N)
- net FS_RX5_P_A is gone; now on net FS_RX5_P: U22.40 (TX5P)
- net FS_RX6_N_A is gone; now on net FS_RX6_N: U22.36 (TX6N)
- net FS_RX6_P_A is gone; now on net FS_RX6_P: U22.37 (TX6P)
- net FS_RX7_N_A is gone; now on net FS_RX7_N: U22.33 (TX7N)
- net FS_RX7_P_A is gone; now on net FS_RX7_P: U22.34 (TX7P)
- net FS_TX0_N_A is gone; now on net FS_TX0_N: U21.2 (RX0N)
- net FS_TX0_P_A is gone; now on net FS_TX0_P: U21.1 (RX0P)
- net FS_TX1_N_A is gone; now on net FS_TX1_N: U21.5 (RX1N)
- net FS_TX1_P_A is gone; now on net FS_TX1_P: U21.4 (RX1P)
- net FS_TX2_N_A is gone; now on net FS_TX2_N: U21.8 (RX2N)
- net FS_TX2_P_A is gone; now on net FS_TX2_P: U21.7 (RX2P)
- net FS_TX3_N_A is gone; now on net FS_TX3_N: U21.11 (RX3N)
- net FS_TX3_P_A is gone; now on net FS_TX3_P: U21.10 (RX3P)
- net FS_TX4_N_A is gone; now on net FS_TX4_N: U22.2 (RX0N)
- net FS_TX4_P_A is gone; now on net FS_TX4_P: U22.1 (RX0P)
- net FS_TX5_N_A is gone; now on net FS_TX5_N: U22.5 (RX1N)
- net FS_TX5_P_A is gone; now on net FS_TX5_P: U22.4 (RX1P)
- net FS_TX6_N_A is gone; now on net FS_TX6_N: U22.8 (RX2N)
- net FS_TX6_P_A is gone; now on net FS_TX6_P: U22.7 (RX2P)
- net FS_TX7_N_A is gone; now on net FS_TX7_N: U22.11 (RX3N)
- net FS_TX7_P_A is gone; now on net FS_TX7_P: U22.10 (RX3P)
- net SATA0_RX_N is gone; now on net GND: J1.B71 (SATA0_RX_N)
- net SATA0_RX_P is gone; now on net FS_RX5_N: J1.B70 (SATA0_RX_P)
- net SATA0_TX_N is gone; now on net GND: J1.A74 (SATA0_TX_N)
- net SATA0_TX_P is gone; now on net FS_TX6_N: J1.A73 (SATA0_TX_P)
- net 12V_MAIN_IN: no longer J12.J1, J12.J10, J12.J11, J12.J12, J12.J2, J12.J3, J12.J4, J12.J5, J12.J6, J12.J7, J12.J8, J12.J9
- net 3V3_SB: now also J1.A93 (VIN_PWR_OK), J1.B93 (UART0_TX), C84.1, J13.J13, J13.J14, J13.J16, J13.J17, R128.2, R129.2, U27.1 (VCCI), U27.16 (VCCP), U27.3 (RESET); no longer J1.B107 (3V3_SB), J1.B108 (3V3_SB)
- net 5V_SBY: now also J1.A94 (GND), J1.A95 (PLTRST#), J1.A96 (THERMTRIP#), J1.B94 (GND), J1.B95 (UART0_RX), J1.B96 (FAN_PWMOUT); no longer J1.A107 (5V_SBY), J1.A108 (5V_SBY), J1.A110 (5V_SBY), J1.A111 (5V_SBY), J1.B110 (5V_SBY), J1.B111 (5V_SBY)
- net CB_CARRIER_HOT_N: now also J1.A89 (SUS_S3#); no longer J1.A98 (CARRIER_HOT#)
- net CB_FAN_PWM: now also J1.B88 (GND); no longer J1.B96 (FAN_PWMOUT)
- net CB_FAN_TACH: now also J1.B89 (BIOS_SEL); no longer J1.B98 (FAN_TACHIN)
- net CB_I2C0_SCL: now also J1.B84 (GND); no longer J1.B90 (I2C0_CLK)
- net CB_I2C0_SDA: now also J1.B85 (GND); no longer J1.B92 (I2C0_DAT)
- net CB_PLTRST_N: now also J1.A87 (FS_PET5_N); no longer J1.A95 (PLTRST#)
- net CB_PWRBTN_N: now also J14.A29 (REFCLK1+); no longer J1.B99 (PWRBTN#)
- net CB_PWR_ALERT_N: now also J1.B91 (GND); no longer J1.A105 (PWR_ALERT#)
- net CB_RSMRST_N: now also J1.A85 (GND); no longer J1.A92 (RSMRST_OUT#)
- net CB_SUS_S3_N: now also J1.A83 (FS_PET4_N); no longer J1.A89 (SUS_S3#)
- net CB_SUS_S45_N: now also J1.A84 (GND); no longer J1.A90 (SUS_S4_S5#)
- net CB_THERMTRIP_N: now also J1.A88 (GND); no longer J1.A96 (THERMTRIP#)
- net CB_UART0_RX: now also J1.B87 (FS_PER5_P); no longer J1.B95 (UART0_RX)
- net CB_UART0_TX: now also J1.B86 (FS_PER5_N); no longer J1.B93 (UART0_TX)
- net CB_VIN_PWR_OK: now also J1.A86 (FS_PET5_P); no longer J1.A93 (VIN_PWR_OK)
- net CB_WAKE_N: now also J1.A90 (SUS_S4_S5#); no longer J1.A99 (WAKE0#)
- net EFUSE_IN: now also J1.A102 (FS_PET6_N), J1.A103 (GND), J1.A104 (RSTBTN#), J1.A105 (PWR_ALERT#), J1.A106 (GND), J1.A107 (5V_SBY), J1.B102 (FS_REFCLK1_N), J1.B103 (GND), J1.B104 (FS_PER6_N), J1.B105 (FS_PER6_P), J1.B106 (GND), J1.B107 (3V3_SB)
- net FP_MCIO_PRSNT_N: no longer U1.47 (GPIO38)
- net FS_MCIO_PRSNT_N: no longer U1.8 (GPIO10)
- net FS_REFCLK1_N: now also J1.B79 (USB2_SPARE_P); no longer J1.B102 (FS_REFCLK1_N)
- net FS_REFCLK1_P: now also J1.B78 (GND); no longer J1.B101 (FS_REFCLK1_P)
- net FS_REFCLK_N: now also J1.A79 (RSVD_HS_A2_P); no longer J1.A71 (FS_REFCLK_N)
- net FS_REFCLK_P: now also J1.A78 (GND); no longer J1.A70 (FS_REFCLK_P)
- net FS_RX0_N: now also J1.B55 (FS_PER7_N); no longer J1.B68 (FS_PER0_N)
- net FS_RX0_P: now also J1.B54 (FS_PER7_P); no longer J1.B67 (FS_PER0_P)
- net FS_RX1_N: now also J1.B58 (FS_PER3_P); no longer J1.B65 (FS_PER1_N)
- net FS_RX1_P: now also J1.B57 (GND); no longer J1.B64 (FS_PER1_P)
- net FS_RX2_N: now also J1.B61 (FS_PER2_P); no longer J1.B62 (FS_PER2_N)
- net FS_RX2_P: now also J1.B60 (GND); no longer J1.B61 (FS_PER2_P)
- net FS_RX3_N: now also J1.B64 (FS_PER1_P); no longer J1.B59 (FS_PER3_N)
- net FS_RX3_P: now also J1.B63 (GND); no longer J1.B58 (FS_PER3_P)
- net FS_RX4_N: now also J1.B67 (FS_PER0_P); no longer J1.B83 (FS_PER4_N)
- net FS_RX4_P: now also J1.B66 (GND); no longer J1.B82 (FS_PER4_P)
- net FS_RX5_N: no longer J1.B86 (FS_PER5_N)
- net FS_RX5_P: now also J1.B69 (GND); no longer J1.B87 (FS_PER5_P)
- net FS_RX6_N: now also J1.B73 (USB2_MCU_P); no longer J1.B104 (FS_PER6_N)
- net FS_RX6_P: now also J1.B72 (GND); no longer J1.B105 (FS_PER6_P)
- net FS_RX7_N: now also J1.B76 (USB2_FACES_P); no longer J1.B55 (FS_PER7_N)
- net FS_RX7_P: now also J1.B75 (GND); no longer J1.B54 (FS_PER7_P)
- net FS_TX0_N: now also J1.A55 (FS_PET7_N); no longer J1.A68 (FS_PET0_N)
- net FS_TX0_P: now also J1.A54 (FS_PET7_P); no longer J1.A67 (FS_PET0_P)
- net FS_TX1_N: now also J1.A58 (FS_PET3_P); no longer J1.A65 (FS_PET1_N)
- net FS_TX1_P: now also J1.A57 (GND); no longer J1.A64 (FS_PET1_P)
- net FS_TX2_N: now also J1.A61 (FS_PET2_P); no longer J1.A62 (FS_PET2_N)
- net FS_TX2_P: now also J1.A60 (GND); no longer J1.A61 (FS_PET2_P)
- net FS_TX3_N: now also J1.A64 (FS_PET1_P); no longer J1.A59 (FS_PET3_N)
- net FS_TX3_P: now also J1.A63 (GND); no longer J1.A58 (FS_PET3_P)
- net FS_TX4_N: now also J1.A67 (FS_PET0_P); no longer J1.A83 (FS_PET4_N)
- net FS_TX4_P: now also J1.A66 (GND); no longer J1.A82 (FS_PET4_P)
- net FS_TX5_N: now also J1.A70 (FS_REFCLK_P); no longer J1.A87 (FS_PET5_N)
- net FS_TX5_P: now also J1.A69 (GND); no longer J1.A86 (FS_PET5_P)
- net FS_TX6_N: no longer J1.A102 (FS_PET6_N)
- net FS_TX6_P: now also J1.A72 (GND); no longer J1.A101 (FS_PET6_P)
- net FS_TX7_N: now also J1.A76 (RSVD_HS_A1_P); no longer J1.A55 (FS_PET7_N)
- net FS_TX7_P: now also J1.A75 (GND); no longer J1.A54 (FS_PET7_P)
- net GND: now also J1.A101 (FS_PET6_P), J1.A108 (5V_SBY), J1.A110 (5V_SBY), J1.A111 (5V_SBY), J1.A59 (FS_PET3_N), J1.A62 (FS_PET2_N), J1.A65 (FS_PET1_N), J1.A68 (FS_PET0_N), J1.A71 (FS_REFCLK_N), J1.A77 (RSVD_HS_A1_N), J1.A80 (RSVD_HS_A2_N), J1.A92 (RSMRST_OUT#), J1.A98 (CARRIER_HOT#), J1.A99 (WAKE0#), J1.B101 (FS_REFCLK1_P), J1.B108 (3V3_SB), J1.B110 (5V_SBY), J1.B111 (5V_SBY), J1.B59 (FS_PER3_N), J1.B62 (FS_PER2_N), J1.B65 (FS_PER1_N), J1.B68 (FS_PER0_N), J1.B74 (USB2_MCU_N), J1.B77 (USB2_FACES_N), J1.B80 (USB2_SPARE_N), J1.B82 (FS_PER4_P), J1.B83 (FS_PER4_N), J1.B90 (I2C0_CLK), J1.B92 (I2C0_DAT), J1.B98 (FAN_TACHIN), J1.B99 (PWRBTN#), J12.J1, J12.J10, J12.J11, J12.J12, J12.J2, J12.J3, J12.J4, J12.J5, J12.J6, J12.J7, J12.J8, J12.J9, C84.2, J13.A12, J13.A15, J13.A18, J13.A2, J13.A21, J13.A24, J13.A27, J13.A28, J13.A29, J13.A3, J13.A6, J13.A9, J13.B12, J13.B15, J13.B18, J13.B21, J13.B24, J13.B27, J13.B28, J13.B3, J13.B6, J13.B9, J13.C12, J13.C15, J13.C18, J13.C21, J13.C24, J13.C27, J13.C28, J13.C3, J13.C6, J13.C9, J13.D10, J13.D11, J13.D12, J13.D13, J13.D14, J13.D15, J13.D16, J13.D17, J13.D18, J13.D19, J13.D2, J13.D20, J13.D21, J13.D22, J13.D23, J13.D24, J13.D25, J13.D26, J13.D27, J13.D28, J13.D29, J13.D3, J13.D4, J13.D5, J13.D6, J13.D7, J13.D8, J13.D9, J13.E12, J13.E15, J13.E18, J13.E21, J13.E24, J13.E27, J13.E28, J13.E3, J13.E6, J13.E9, J13.F12, J13.F15, J13.F18, J13.F21, J13.F24, J13.F27, J13.F28, J13.F3, J13.F6, J13.F9, J13.G10, J13.G11, J13.G12, J13.G13, J13.G14, J13.G15, J13.G16, J13.G17, J13.G18, J13.G19, J13.G2, J13.G20, J13.G21, J13.G22, J13.G23, J13.G24, J13.G25, J13.G26, J13.G27, J13.G28, J13.G29, J13.G3, J13.G4, J13.G5, J13.G6, J13.G7, J13.G8, J13.G9, J13.H12, J13.H15, J13.H18, J13.H21, J13.H24, J13.H27, J13.H28, J13.H3, J13.H6, J13.H9, J13.I12, J13.I15, J13.I18, J13.I21, J13.I24, J13.I27, J13.I28, J13.I3, J13.I6, J13.I9, J13.J12, J13.J15, J13.J18, J13.J2, J13.J21, J13.J24, J13.J27, J13.J28, J13.J29, J13.J3, J13.J6, J13.J9, J14.A1 (GND), J14.A10 (GND), J14.A12 (REFCLK-), J14.A13 (GND), J14.A16 (GND), J14.A19 (GND), J14.A22 (GND), J14.A25 (GND), J14.A28 (GND), J14.A30 (REFCLK1-), J14.A31 (GND), J14.A34 (GND), J14.A37 (GND), J14.A38 (GND), J14.A4 (GND), J14.A41 (GND), J14.A44 (GND), J14.A47 (GND), J14.A50 (GND), J14.A53 (GND), J14.A54 (PER13P), J14.A55 (PER13N), J14.A56 (GND), J14.A57 (PER14P), J14.A58 (PER14N), J14.A59 (GND), J14.A60 (PER15P), J14.A61 (PER15N), J14.A62 (GND), J14.A7 (GND), J14.B1 (GND), J14.B10 (GND), J14.B13 (GND), J14.B16 (GND), J14.B19 (GND), J14.B22 (GND), J14.B25 (GND), J14.B28 (GND), J14.B30 (PRSNT1), J14.B31 (GND), J14.B34 (GND), J14.B37 (GND), J14.B38 (GND), J14.B4 (GND), J14.B41 (GND), J14.B44 (GND), J14.B47 (GND), J14.B50 (GND), J14.B53 (GND), J14.B54 (PET13P), J14.B55 (PET13N), J14.B56 (GND), J14.B57 (PET14P), J14.B58 (PET14N), J14.B59 (GND), J14.B60 (PET15P), J14.B61 (PET15N), J14.B62 (GND), J14.B7 (GND), J14.MP (SHIELD), R127.2, U27.2 (ADDR), U27.8 (GND); no longer J1.A103 (GND), J1.A106 (GND), J1.A57 (GND), J1.A60 (GND), J1.A63 (GND), J1.A66 (GND), J1.A69 (GND), J1.A72 (GND), J1.A75 (GND), J1.A78 (GND), J1.A81 (GND), J1.A84 (GND), J1.A85 (GND), J1.A88 (GND), J1.A91 (GND), J1.A94 (GND), J1.B103 (GND), J1.B106 (GND), J1.B57 (GND), J1.B60 (GND), J1.B63 (GND), J1.B66 (GND), J1.B69 (GND), J1.B72 (GND), J1.B75 (GND), J1.B78 (GND), J1.B84 (GND), J1.B85 (GND), J1.B88 (GND), J1.B91 (GND), J1.B94 (GND)
- net HALL_A_N: now also J13.J10
- net HALL_B_N: now also J13.J11
- net I2C_SYS_SCL: now also J13.H2, J13.J19, U27.14 (SCL)
- net I2C_SYS_SDA: now also J13.I2, J13.J20, U27.15 (SDA)
- net IOB_PRSNT_N: now also J13.H29
- net PWRBTN_IN_N: now also J13.C29
- net SYS_INT_N: now also J13.B29, J13.J22
- net USB2_FACES_N: no longer J1.B77 (USB2_FACES_N)
- net USB2_FACES_P: no longer J1.B76 (USB2_FACES_P)
- net USB2_MCU_N: now also J1.A82 (FS_PET4_P); no longer J1.B74 (USB2_MCU_N)
- net USB2_MCU_P: now also J1.A81 (GND); no longer J1.B73 (USB2_MCU_P)
- net USB2_SPARE_N: now also J13.J8; no longer J1.B80 (USB2_SPARE_N)
- net USB2_SPARE_P: now also J13.J7; no longer J1.B79 (USB2_SPARE_P)
- net PSU_PWR_OK_M renamed CB_SMB_ALERT_N
- net CB_SMB_ALERT_N: now also J14.B29 (PERST1)
- new net I2C_BB_SCL: J14.B26 (RSVD), U1.47 (GPIO38)
- new net I2C_BB_SDA: J14.B27 (RSVD), U1.8 (GPIO10)
- new net IOB_ACT_LED: J13.F29, U27.9 (P4)
- new net IOB_ASM_CLKREQ_N: J13.I1, J14.B8 (SMCLK)
- new net IOB_ASM_PERST_N: J13.H1, J14.A11 (REFCLK+)
- new net IOB_ASM_PERX0_N: J13.E17, J14.B33 (PET6N)
- new net IOB_ASM_PERX0_P: J13.E16, J14.B32 (PET6P)
- new net IOB_ASM_PERX1_N: J13.E20, J14.B36 (PET7N)
- new net IOB_ASM_PERX1_P: J13.E19, J14.B35 (PET7P)
- new net IOB_ASM_PERX2_N: J13.E23, J14.B40 (PET8N)
- new net IOB_ASM_PERX2_P: J13.E22, J14.B39 (PET8P)
- new net IOB_ASM_PERX3_N: J13.E26, J14.B43 (PET9N)
- new net IOB_ASM_PERX3_P: J13.E25, J14.B42 (PET9P)
- new net IOB_ASM_PETX0_N: J13.E5, J14.A33 (PER6N)
- new net IOB_ASM_PETX0_P: J13.E4, J14.A32 (PER6P)
- new net IOB_ASM_PETX1_N: J13.E8, J14.A36 (PER7N)
- new net IOB_ASM_PETX1_P: J13.E7, J14.A35 (PER7P)
- new net IOB_ASM_PETX2_N: J13.E11, J14.A40 (PER8N)
- new net IOB_ASM_PETX2_P: J13.E10, J14.A39 (PER8P)
- new net IOB_ASM_PETX3_N: J13.E14, J14.A43 (PER9N)
- new net IOB_ASM_PETX3_P: J13.E13, J14.A42 (PER9P)
- new net IOB_ASM_REFCLK_N: J13.F5, J14.B24 (PET5N)
- new net IOB_ASM_REFCLK_P: J13.F4, J14.B23 (PET5P)
- new net IOB_DPA_AUX_N: J13.A17
- new net IOB_DPA_AUX_P: J13.A16
- new net IOB_DPA_HPD: J13.A1
- new net IOB_DPA_ML0_N: J13.A5
- new net IOB_DPA_ML0_P: J13.A4
- new net IOB_DPA_ML1_N: J13.A8
- new net IOB_DPA_ML1_P: J13.A7
- new net IOB_DPA_ML2_N: J13.A11
- new net IOB_DPA_ML2_P: J13.A10
- new net IOB_DPA_ML3_N: J13.A14
- new net IOB_DPA_ML3_P: J13.A13
- new net IOB_DPB_AUX_N: J13.B8
- new net IOB_DPB_AUX_P: J13.B7
- new net IOB_DPB_HPD: J13.B1
- new net IOB_DPB_ML0_N: J13.A20
- new net IOB_DPB_ML0_P: J13.A19
- new net IOB_DPB_ML1_N: J13.A23
- new net IOB_DPB_ML1_P: J13.A22
- new net IOB_DPB_ML2_N: J13.A26
- new net IOB_DPB_ML2_P: J13.A25
- new net IOB_DPB_ML3_N: J13.B5
- new net IOB_DPB_ML3_P: J13.B4
- new net IOB_DPC_AUX_N: J13.B23
- new net IOB_DPC_AUX_P: J13.B22
- new net IOB_DPC_HPD: J13.C1
- new net IOB_DPC_ML0_N: J13.B11
- new net IOB_DPC_ML0_P: J13.B10
- new net IOB_DPC_ML1_N: J13.B14
- new net IOB_DPC_ML1_P: J13.B13
- new net IOB_DPC_ML2_N: J13.B17
- new net IOB_DPC_ML2_P: J13.B16
- new net IOB_DPC_ML3_N: J13.B20
- new net IOB_DPC_ML3_P: J13.B19
- new net IOB_DPD_AUX_N: J13.C14
- new net IOB_DPD_AUX_P: J13.C13
- new net IOB_DPD_HPD: J13.G1
- new net IOB_DPD_ML0_N: J13.B26
- new net IOB_DPD_ML0_P: J13.B25
- new net IOB_DPD_ML1_N: J13.C5
- new net IOB_DPD_ML1_P: J13.C4
- new net IOB_DPD_ML2_N: J13.C8
- new net IOB_DPD_ML2_P: J13.C7
- new net IOB_DPD_ML3_N: J13.C11
- new net IOB_DPD_ML3_P: J13.C10
- new net IOB_HDMI_CEC: J13.F1
- new net IOB_HDMI_DDC_SCL: J13.D1
- new net IOB_HDMI_DDC_SDA: J13.E1
- new net IOB_LAN1_CLKREQ_N: J13.B2, J14.B11 (PERST)
- new net IOB_LAN1_PERST_N: J13.J1, J14.A26 (CLKREQ1)
- new net IOB_LAN1_PERX_N: J13.F11, J14.B46 (PET10N)
- new net IOB_LAN1_PERX_P: J13.F10, J14.B45 (PET10P)
- new net IOB_LAN1_PETX_N: J13.F8, J14.A46 (PER10N)
- new net IOB_LAN1_PETX_P: J13.F7, J14.A45 (PER10P)
- new net IOB_LAN1_REFCLK_N: J13.F14, J14.A24 (PER5N)
- new net IOB_LAN1_REFCLK_P: J13.F13, J14.A23 (PER5P)
- new net IOB_LAN2_CLKREQ_N: J13.E2, J14.B12 (PRSNT)
- new net IOB_LAN2_PERST_N: J13.C2, J14.A27 (WAKE1)
- new net IOB_LAN2_PERX_N: J13.F20, J14.B52 (PET12N)
- new net IOB_LAN2_PERX_P: J13.F19, J14.B51 (PET12P)
- new net IOB_LAN2_PETX_N: J13.F17, J14.A52 (PER12N)
- new net IOB_LAN2_PETX_P: J13.F16, J14.A51 (PER12P)
- new net IOB_LAN2_REFCLK_N: J13.F23, J14.B49 (PET11N)
- new net IOB_LAN2_REFCLK_P: J13.F22, J14.B48 (PET11P)
- new net IOB_PCIE_WAKE_N: J13.F2, J14.B9 (SMDAT)
- new net IOB_PLT_RST_N: J13.B30, R127.1, U27.4 (P0)
- new net IOB_PWR_LED: J13.E29, U27.7 (P3)
- new net IOB_SLP_S3_N: J13.I29, J14.A8 (CLKREQ)
- new net IOB_SLP_S5_N: J13.A30, J14.A9 (WAKE)
- new net IOB_USB2_1_N: J13.I11
- new net IOB_USB2_1_P: J13.I10
- new net IOB_USB2_2_N: J13.I14
- new net IOB_USB2_2_P: J13.I13
- new net IOB_USB2_3_N: J13.I17
- new net IOB_USB2_3_P: J13.I16
- new net IOB_USB2_4_N: J13.I20
- new net IOB_USB2_4_P: J13.I19
- new net IOB_USB2_5_N: J13.I23
- new net IOB_USB2_5_P: J13.I22
- new net IOB_USB2_6_N: J13.I26
- new net IOB_USB2_6_P: J13.I25
- new net IOB_USB2_7_N: J13.J5
- new net IOB_USB2_7_P: J13.J4
- new net IOB_USB3_1_RX_N: J13.H8, J14.B3 (PET0N)
- new net IOB_USB3_1_RX_P: J13.H7, J14.B2 (PET0P)
- new net IOB_USB3_1_TX_N: J13.H5, J14.A3 (PER0N)
- new net IOB_USB3_1_TX_P: J13.H4, J14.A2 (PER0P)
- new net IOB_USB3_2_RX_N: J13.H14, J14.B6 (PET1N)
- new net IOB_USB3_2_RX_P: J13.H13, J14.B5 (PET1P)
- new net IOB_USB3_2_TX_N: J13.H11, J14.A6 (PER1N)
- new net IOB_USB3_2_TX_P: J13.H10, J14.A5 (PER1P)
- new net IOB_USB3_3_RX_N: J13.H20, J14.B15 (PET2N)
- new net IOB_USB3_3_RX_P: J13.H19, J14.B14 (PET2P)
- new net IOB_USB3_3_TX_N: J13.H17, J14.A15 (PER2N)
- new net IOB_USB3_3_TX_P: J13.H16, J14.A14 (PER2P)
- new net IOB_USB3_4_RX_N: J13.H26, J14.B21 (PET4N)
- new net IOB_USB3_4_RX_P: J13.H25, J14.B20 (PET4P)
- new net IOB_USB3_4_TX_N: J13.H23, J14.A21 (PER4N)
- new net IOB_USB3_4_TX_P: J13.H22, J14.A20 (PER4P)
- new net IOB_USB3_5_RX_N: J13.I8, J14.B18 (PET3N)
- new net IOB_USB3_5_RX_P: J13.I7, J14.B17 (PET3P)
- new net IOB_USB3_5_TX_N: J13.I5, J14.A18 (PER3N)
- new net IOB_USB3_5_TX_P: J13.I4, J14.A17 (PER3P)
- new net IOB_USB_OC_N_A: J13.D30, R128.1, U27.5 (P1)
- new net IOB_USB_OC_N_C: J13.C30, R129.1, U27.6 (P2)
- new net USB2_HUB_UP_N: J14.A49 (PER11N)
- new net USB2_HUB_UP_P: J14.A48 (PER11P)
- no-connect marks 474 -> 402
Other:
- note added: "Gen5 redrivers (Aidan 2026-10-28): U20 DS320PR1601 GPU x16 (A side = J1/CPU, B side = GPU face), U21/U22 DS320PR810 SSD x8 (FS lanes 0-3 / 4-7). No NDA parts (Aidan 2026-10-29). High-speed nets *_A / *_B are NOT yet spliced into FP_*/FS_* (J1->J9/J10 copper still direct): net split + reroute pending. 3V3_RDRV is a NEW rail, source TBD (~10.5 W max = 3.2 A @3.3 V; 3V3_SB buck is 3 A standby, not u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"
- note removed: "Gen5 redrivers (Aidan 2026-10-28): U20 DS320PR1601 GPU x16 (A side = J1/CPU, B side = GPU face), U21/U22 DS320PR810 SSD x8 (FS lanes 0-3 / 4-7), U23 PT5161L fallback DNP (no pins, NDA, NOT pin-compatible-assumed). High-speed nets *_A / *_B are NOT yet spliced into FP_*/FS_* (J1->J9/J10 copper still direct): net split + reroute pending. 3V3_RDRV is a NEW rail, source TBD (~10.5 W max = 3.2 A @3.3 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"
