File: boards/cpu-am5/kicad/macpro62_am5_v4.kicad_pcb (KiCad board)
At the start: 10 copper layers, 156 x 167.8 mm, 57 parts, among them J1 J1 CPU-LINK 224 fingers (AM5 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, J3 J3 IOB-HS MCIO 124 RA (AM5 ho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, J4 J4 SPI TPM (opt.), J5 J5 debug UART/SWD/POST, J8 J8 M.2 2280 boot (PROM21 Gen4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, Q1 PS VDDCR 1 SiC654, Q2 PS VDDCR 2 SiC654, Q3 PS VDDCR 3 SiC654, Q4 PS VDDCR 4 SiC654, Q5 PS VDDCR 5 SiC654, Q6 PS SOC 1 SiC654, Q7 PS SOC 2 SiC654, Q8 PS MISC SiC654, U1 U1 Socket AM5 LGA1718 PLACEHO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, U10 U10 FCH SPI 32MB (Dasharo), U11 U11 eFuse 12V IN (whole CB), U14 U14 ALC897 DNP (FCH AZ), U15 U15 INA228 + RS1 0.5 mOhm (12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, U16 U16 VL822-Q7 USB 10G hub (J3 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, U17 U17 PROM21 SPI flash, U2 U2 PROM21 218-0891025 PLACEHO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, U3 U3 SVI3 3-rail ctrl RAA229139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, U4 CPU S5/aux rails (1.8/3.3/MIS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, U5 CPU seq/straps/SVI3 pull-ups, U6 PROM21 rails, U7 5V VIN_BULK 4x UDIMM, U8 VDDIO_MEM_S3 1.1V, U9 U9 EC RP2350, Y1 Y1/Y2 48M + 32k (FCH)

Commit message: Sync design state 2026-10-29: J1 v4 pinned, boot drive dropped, no NDA parts, base board J13/J14 and fab push, SSD/I/O power and pinmaps
Changed lines of the file:
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@@
 			)
 		)
-		(pad "1" thru_hole circle
+		(pad "1" thru_hole oval
 			(at 0 0)
-			(size 9 9)
-			(drill 5)
+			(size 10 9)
+			(drill oval 6 5)
 			(layers "*.Cu" "*.Mask")
 			(remove_unused_layers no)
